Commit message: working

File: alphaDroneClean/fly_boy/fly_boy.urdf (robot description, URDF)
Before this commit: robot quadrotor, 5 links, 4 joints
Joints:
- joint rotor_1_joint: limit lower=0 upper=1000 effort=1.0 velocity=1000 -> effort=0.01 velocity=1000; type revolute -> continuous
- joint rotor_2_joint: limit lower=0 upper=1000 effort=1.0 velocity=1000 -> effort=0.01 velocity=1000; type revolute -> continuous
- joint rotor_3_joint: limit lower=0 upper=1000 effort=1.0 velocity=1000 -> effort=0.01 velocity=1000; type revolute -> continuous
- joint rotor_4_joint: limit lower=0 upper=1000 effort=1.0 velocity=1000 -> effort=0.01 velocity=1000; type revolute -> continuous
