Commit message: new model

File: alphaDroneClean/assets/fly_boy/fly_boy.urdf (robot description, URDF)
Before this commit: robot quadrotor, 5 links, 4 joints
Links:
- link base_link: mass 3.683 -> 3.866
Joints:
- joint rotor_1_joint: origin xyz=0.197 -0.22465 0.025 rpy=0 0 0 -> xyz=0.208 -0.22465 0.025 rpy=0 0 0
- joint rotor_2_joint: origin xyz=0.197 0.22465 0.025 rpy=0 0 0 -> xyz=0.208 0.22465 0.025 rpy=0 0 0
- joint rotor_3_joint: origin xyz=-0.217 0.22465 0.025 rpy=0 0 0 -> xyz=-0.228 0.22465 0.025 rpy=0 0 0
- joint rotor_4_joint: origin xyz=-0.217 -0.22465 0.025 rpy=0 0 0 -> xyz=-0.228 -0.22465 0.025 rpy=0 0 0

Commit message: iavdbkhbkjbsadkj b

File: alphaDroneClean/assets/fly_boy/fly_boy.urdf (robot description, URDF)
Before this commit: robot quadrotor, 5 links, 4 joints
Links:
- link base_link: mass 3.866 -> 3.833
- link rotor_1: mass 0.05 -> 0.0001
- link rotor_2: mass 0.05 -> 0.0001
- link rotor_3: mass 0.05 -> 0.0001
- link rotor_4: mass 0.05 -> 0.0001
